Commit message: Inegration of depth camera

File: robot/description/robot.urdf.xacro (robot description, xacro)
@@ -4,4 +4,5 @@
     <xacro:include filename="gazebo_control.xacro" />
     <xacro:include filename="lidar.xacro" />
-    <xacro:include filename="camera.xacro" />
+    <!-- <xacro:include filename="camera.xacro" />   -->
+    <xacro:include filename="depth_camera.xacro" />
 </robot>

File: robot/description/robot_core.xacro (robot description, xacro)
@@ -13,4 +13,7 @@
     <material name="black">
         <color rgba="0 0 0 1"/>
+    </material>
+    <material name="red">
+        <color rgba="1 0 0 1"/>
     </material>
     <!-- BASE LINK -->
